Commit message: -Start turtlebot in sick robot day world per default

File: hector_turtlebot_description/urdf/turtlebot_sick_setup.xacro (robot description, xacro)
@@ -14,3 +14,6 @@
     <origin xyz="-0.115 0.0 0.06" rpy="0 0 0"/>
   </xacro:hokuyo_utm30lx>
+<!--  <xacro:hokuyo_utm30lx name="hokuyo_laser" parent="base_link" ros_topic="hokuyo_scan" update_rate="40" ray_count="1040" min_angle="130" max_angle="-130">
+    <origin xyz="-0.115 0.0 0.26" rpy="0 0 0"/>
+  </xacro:hokuyo_utm30lx>-->
 </robot>

Commit message: -Add asus xtion cam for the moment

File: hector_turtlebot_description/urdf/turtlebot_sick_setup.xacro (robot description, xacro)
@@ -11,4 +11,5 @@
   <!--<sensor_kinect  parent="base_link"/>-->
   <xacro:include filename="$(find hector_sensors_description)/urdf/hokuyo_utm30lx.urdf.xacro" />
+  <xacro:include filename="$(find hector_sensors_description)/urdf/asus_camera.urdf.xacro" />
   <xacro:hokuyo_utm30lx name="hokuyo_laser" parent="plate_2_link" ros_topic="hokuyo_scan" update_rate="40" ray_count="1040" min_angle="130" max_angle="-130">
     <origin xyz="-0.115 0.0 0.06" rpy="0 0 0"/>
@@ -17,3 +18,6 @@
     <origin xyz="-0.115 0.0 0.26" rpy="0 0 0"/>
   </xacro:hokuyo_utm30lx>-->
+  <xacro:asus_camera name="openni" parent="base_link">
+    <origin xyz="0 0  0.45" rpy="0 0 0"/>
+  </xacro:asus_camera>
 </robot>

Commit message: -Add camera xacro file for working around the fact that generic camera plugin doesn´t work in hydro -Add cameras as mounted on real system

File: hector_turtlebot_description/urdf/turtlebot_sick_setup.xacro (robot description, xacro)
@@ -8,16 +8,26 @@
   <xacro:include filename="$(find turtlebot_description)/urdf/turtlebot_library.urdf.xacro" />
   <create/>
-  <stack_circles parent="base_link"/>
+  <!--<stack_circles parent="base_link"/>-->
   <!--<sensor_kinect  parent="base_link"/>-->
   <xacro:include filename="$(find hector_sensors_description)/urdf/hokuyo_utm30lx.urdf.xacro" />
   <xacro:include filename="$(find hector_sensors_description)/urdf/asus_camera.urdf.xacro" />
-  <xacro:hokuyo_utm30lx name="hokuyo_laser" parent="plate_2_link" ros_topic="hokuyo_scan" update_rate="40" ray_count="1040" min_angle="130" max_angle="-130">
-    <origin xyz="-0.115 0.0 0.06" rpy="0 0 0"/>
+  <!--<xacro:include filename="$(find hector_sensors_description)/urdf/generic_camera.urdf.xacro" />-->
+  <xacro:include filename="$(find hector_turtlebot_description)/urdf/camera.urdf.xacro" />
+  <xacro:hokuyo_utm30lx name="hokuyo_laser" parent="base_link" ros_topic="hokuyo_scan" update_rate="40" ray_count="1040" min_angle="130" max_angle="-130">
+    <origin xyz="0.0925 -0.004 0.198" rpy="0 0 0"/>
   </xacro:hokuyo_utm30lx>
-<!--  <xacro:hokuyo_utm30lx name="hokuyo_laser" parent="base_link" ros_topic="hokuyo_scan" update_rate="40" ray_count="1040" min_angle="130" max_angle="-130">
-    <origin xyz="-0.115 0.0 0.26" rpy="0 0 0"/>
-  </xacro:hokuyo_utm30lx>-->
-  <xacro:asus_camera name="openni" parent="base_link">
-    <origin xyz="0 0  0.45" rpy="0 0 0"/>
+  <xacro:asus_camera name="camera" parent="base_link">
+    <origin xyz="0.07 0.10  0.3" rpy="0 -0.30 0.872664626"/>
   </xacro:asus_camera>
+  <xacro:generic_camera name="forward_cam" parent="base_link">
+    <origin xyz="0.1595 0.0 0.22" rpy="0 0 0"/>
+  </xacro:generic_camera>
+  <!--
+  <xacro:generic_camera name="forward_cam" parent="base_link" ros_topic="image_raw" cam_info_topic="camera_info" update_rate="10" res_x="640" res_y="480" image_format="R8G8B8" hfov="60">
+    <origin xyz="0.1595 0.0 0.22" rpy="0 0 0"/>
+  </xacro:generic_camera>
+  <xacro:asus_camera name="forward_cam" parent="base_link">
+    <origin xyz="0.1595 0.0 0.22" rpy="0 0 0"/>
+  </xacro:asus_camera>
+  -->
 </robot>

Commit message: moved position of asus xtion

File: hector_turtlebot_description/urdf/turtlebot_sick_setup.xacro (robot description, xacro)
@@ -18,5 +18,5 @@
   </xacro:hokuyo_utm30lx>
   <xacro:asus_camera name="camera" parent="base_link">
-    <origin xyz="0.07 0.10  0.3" rpy="0 -0.30 0.872664626"/>
+    <origin xyz="-0.10 0.16  0.3" rpy="0 -0.30 1.65806278939"/>
   </xacro:asus_camera>
   <xacro:generic_camera name="forward_cam" parent="base_link">
